Commit message: Added a new message filter node for left, center and right cameras

File: prius_description/urdf/prius.urdf (robot description, URDF)
Before this commit: robot prius, 24 links, 23 joints
Joints:
- joint left_camera_joint: origin xyz=1 -0.7 1.0 rpy=0 0.05 1.0 -> xyz=1 -0.7 1.0 rpy=0 0.05 -1.5707
- joint right_camera_joint: origin xyz=-1 -0.7 1.0 rpy=0 0.05 2.1416 -> xyz=-1 -0.7 1.0 rpy=0 0.05 -1.5707

Commit message: added a launch file used for recording bag files and updated locations of left and right cams

File: prius_description/urdf/prius.urdf (robot description, URDF)
Before this commit: robot prius, 24 links, 23 joints
Joints:
- joint left_camera_joint: origin xyz=1 -0.7 1.0 rpy=0 0.05 -1.5707 -> xyz=1 -0.65 1.4 rpy=0 0.05 -1.5707
- joint right_camera_joint: origin xyz=-1 -0.7 1.0 rpy=0 0.05 -1.5707 -> xyz=-1 -0.65 1.4 rpy=0 0.05 -1.5707

Commit message: Added a 0.27 rad offset for left and right camera from the center cam

File: prius_description/urdf/prius.urdf (robot description, URDF)
Before this commit: robot prius, 24 links, 23 joints
Joints:
- joint left_camera_joint: origin xyz=1 -0.65 1.4 rpy=0 0.05 -1.5707 -> xyz=1 -0.65 1.4 rpy=0 0.05 -1.3007
- joint right_camera_joint: origin xyz=-1 -0.65 1.4 rpy=0 0.05 -1.5707 -> xyz=-1 -0.65 1.4 rpy=0 0.05 -1.8407
